Commit message: Lidar adjustments

File: description/lidar.xacro (robot description, xacro)
@@ -4,5 +4,5 @@
         <parent link="chassis"/>
         <child link="laser_frame"/>
-        <origin xyz="0.122 0 0.212" rpy="0 0 0"/>
+        <origin xyz="0.122 0 0.127" rpy="0 0 0"/>
     </joint>
     <link name="laser_frame">

Commit message: Reshaping Lidar and positioning

File: description/lidar.xacro (robot description, xacro)
@@ -4,10 +4,10 @@
         <parent link="chassis"/>
         <child link="laser_frame"/>
-        <origin xyz="0.122 0 0.127" rpy="0 0 0"/>
+        <origin xyz="0.0381 0 0.127" rpy="0 0 0"/>
     </joint>
     <link name="laser_frame">
         <visual>
             <geometry>
-                <cylinder radius="0.05" length="0.04"/>
+                <cylinder radius="0.0349" length="0.04"/>
             </geometry>
             <material name="black"/>
@@ -22,5 +22,5 @@
         <collision>
             <geometry>
-                <cylinder radius="0.05" length="0.04"/>
+                <cylinder radius="0.0349" length="0.04"/>
             </geometry>
         </collision>
