Commit message: Final Thoughts

File: description/camera.xacro (robot description, xacro)
@@ -4,5 +4,5 @@
         <parent link="chassis"/>
         <child link="camera_link"/>
-        <origin xyz="0.276 0 0.181" rpy="0 0.18 0"/>
+        <origin xyz="0.276 0 0.081" rpy="0 0.18 0"/>
     </joint>
     <link name="camera_link">
@@ -16,5 +16,5 @@
             <origin xyz="0 0 -0.05"/>
             <geometry>
-                <cylinder radius="0.002" length="0.1"/>
+                <cylinder radius="0.002" length="0.075"/>
             </geometry>
             <material name="black"/>

File: description/lidar.xacro (robot description, xacro)
@@ -4,17 +4,17 @@
         <parent link="chassis"/>
         <child link="laser_frame"/>
-        <origin xyz="0.0381 0 0.127" rpy="0 0 0"/>
+        <origin xyz="0.0381 0 0.05" rpy="0 0 0"/>
     </joint>
     <link name="laser_frame">
         <visual>
             <geometry>
-                <cylinder radius="0.0349" length="0.04"/>
+                <cylinder radius="0.0349" length="0.0254"/>
             </geometry>
             <material name="black"/>
         </visual>
         <visual>
-            <origin xyz="0 0 -0.05"/>
+            <origin xyz="0 0 -0.025"/>
             <geometry>
-                <cylinder radius="0.01" length="0.1"/>
+                <cylinder radius="0.01" length="0.05"/>
             </geometry>
             <material name="black"/>

File: description/robot_core.xacro (robot description, xacro)
@@ -4,5 +4,5 @@
     <xacro:property name="chassis_length" value="0.3048"/>
     <xacro:property name="chassis_width" value="0.3048"/>
-    <xacro:property name="chassis_height" value="0.100"/>
+    <xacro:property name="chassis_height" value="0.010"/>
     <xacro:property name="chassis_mass" value="1.0"/>
     <xacro:property name="wheel_radius" value="0.033"/>
